File: EiMS.kicad_pcb (KiCad board)
At the start: 4 copper layers, 200 x 123 mm, 60 parts, among them J1 Conn_01x06, J2 AudioJack2, J3 AudioJack2, SW1 SW_SPDT, U1 PIC32MM0064GPL028-I_SP, U2 LTC3124, U3 LMC662, U4 IFJM-001, U5 IFJM-001

Commit message: final
Parts:
- added D1: D, Diode_THT:D_A-405_P10.16mm_Horizontal, F.Cu at (93.7, 76.0)
- added D2: D, Diode_THT:D_A-405_P10.16mm_Horizontal, F.Cu at (98.9, 76.0)
- REF1, REF2, REF3, REF4: value MountingHole_2.2mm_M2_ISO7380_Pad -> MountingHole_3.2mm_M3_Pad; footprint MountingHole:MountingHole_2.2mm_M2_ISO7380_Pad -> MountingHole:MountingHole_3.2mm_M3_Pad
- moved REF1 192.1 mm to (239.1, 37.9)
- moved REF2 192.1 mm to (239.1, 153.1)
- moved REF3 192.1 mm to (46.9, 153.1)
- moved REF4 192.1 mm to (46.9, 37.9)
- moved G*** 20.0 mm to (90.0, 48.8)
- moved C2 17.4 mm to (111.0, 64.7), turned to 270 degrees
- moved PS1 12.2 mm to (140.1, 80.0)
- moved PS2 8.49 mm to (100.9, 65.4)
- moved A1 5.13 mm to (52.0, 97.7)
- moved BT1 3.99 mm to (157.3, 52.7)
- moved C4 3.75 mm to (111.0, 74.9), turned to 270 degrees
- moved U3 0.76 mm to (105.3, 114.3)
- moved R7 0.47 mm to (100.2, 118.1)
- moved R3 0.15 mm to (97.1, 92.2)
- moved R4 0.15 mm to (89.4, 96.3)
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Connections:
- SW1 pad 1: Net-(SW1-Pad1) -> Net-(PS1-Pad22)
- SW1 pad 2: Net-(PS1-Pad22) -> Net-(SW1-Pad2)
- U1 pad 14: Net-(U1-Pad14) -> Net-(D2-Pad1)
- U1 pad 15: Net-(U1-Pad15) -> Net-(D1-Pad1)
- U2 pad 6: Net-(PS1-Pad22) -> Net-(SW1-Pad2)
- U4 pad 5: Net-(U1-Pad15) -> Net-(D1-Pad2)
- U4 pad 7: Net-(SW1-Pad1) -> Net-(PS1-Pad22)
- U5 pad 5: Net-(U1-Pad14) -> Net-(D2-Pad2)
- U5 pad 7: Net-(SW1-Pad1) -> Net-(PS1-Pad22)
Routing:
- net Net-(U1-Pad14): track 146.4 -> 0.00 mm
- net Net-(U1-Pad15): track 109.1 -> 0.00 mm
- net Net-(D2-Pad2): track 0.00 -> 81.5 mm
- net Net-(D2-Pad1): track 0.00 -> 57.5 mm
- net Net-(D1-Pad1): track 0.00 -> 52.2 mm
- net Net-(D1-Pad2): track 0.00 -> 49.9 mm
- net Net-(A1-Pad16): track 107.7 -> 77.3 mm
- net Net-(A1-Pad21): track 30.3 -> 19.8 mm, vias 25 -> 24
- net Net-(A1-Pad14): track 71.3 -> 61.8 mm
- net Net-(A1-Pad15): track 82.0 -> 89.6 mm
- net Net-(F2-Pad2): track 14.7 -> 7.67 mm
- net Net-(F2-Pad1): track 38.3 -> 31.3 mm
- net Net-(F1-Pad2): track 14.7 -> 7.67 mm
- net Net-(F1-Pad1): track 38.3 -> 31.3 mm
- net Net-(A1-Pad10): track 66.3 -> 59.4 mm
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- added copper zone on In2.Cu, net Net-(SW1-Pad2)
- removed copper zone on In2.Cu, net Net-(SW1-Pad1)
Other:
- board text added: "Board for “EiMS Device” TEST-Type - Ver. 1.1 Power Supply — 12V, ±5V, 3.7V & 3.3V Max. Voltage of Stimu. — ±60V Max. Ampere of Stimu. — 0.062A Layer — 4layers Thickness — 1.6mm Dimensions — 200mm X 123mm Surface Finish — HASL Lead Free Copper Weight — 1oz Inspired from “wavEMS” Designed by Hiroki Ohara Created in 2021"
- board text removed: "Board for “EiMS Device” TEST-Type - Ver. 1.0 —————————————————————————————— Size: 200 mm x 123 mm x 1.6 mm Power Supply: 12V, 3.7V, 3.3V & ±5V Max. Performance: ±60V, ≈60mA & ≈5,000Hz Inspired from “wavEMS” Designed by Hiroki Ohara Created in 2021 Copyright © 2021 Hiroki Ohara"
