File: DualEMS_PCB.sch (KiCad schematic (older format))
At the start: 57 parts, among them J1 Conn_01x06, J2 AudioJack2, J3 AudioJack2, SW1 SW_SPDT, U1 PIC32MM0064GPL028-I_SP, U2 LTC3124, U3 LMC662, U4 IFJM-001, U5 IFJM-001

Commit message: changed name
Parts:
- A1: footprint EiMS:RN52 -> DualEMS_PCB:RN52; symbol EiMS:RN52 -> DualEMS_PCB:RN52
- BT1: footprint EiMS:Battery_+3V7 -> DualEMS_PCB:Battery_+3V7
- J2, J3: footprint EiMS:MJ-352 -> DualEMS_PCB:MJ-352
- PS1: footprint EiMS:MIWI06-24D05 -> DualEMS_PCB:MIWI06-24D05; symbol EiMS:MIWI06-24D05 -> DualEMS_PCB:MIWI06-24D05
- PS2: footprint EiMS:M78AR033-0.5 -> DualEMS_PCB:M78AR033-0.5; symbol EiMS:M78AR033-0.5 -> DualEMS_PCB:M78AR033-0.5
- U1: footprint EiMS:PIC32MM0064GPL028-I_SP -> DualEMS_PCB:PIC32MM0064GPL028-I_SP; symbol EiMS:PIC32MM0064GPL028-I_SP -> DualEMS_PCB:PIC32MM0064GPL028-I_SP
- U2: footprint EiMS:LTC3124 -> DualEMS_PCB:LTC3124; symbol EiMS:LTC3124 -> DualEMS_PCB:LTC3124
- U3: footprint EiMS:LMC662 -> DualEMS_PCB:LMC662; symbol EiMS:LMC662 -> DualEMS_PCB:LMC662
- U4, U5: footprint EiMS:IFJM-001 -> DualEMS_PCB:IFJM-001; symbol EiMS:IFJM-001 -> DualEMS_PCB:IFJM-001
Changed lines of the file:
@@
 $EndComp
 $Comp
-L EiMS:RN52 A1
+L DualEMS_PCB:RN52 A1
 U 1 1 606F37D4
 P 4250 5650
 F 0 "A1" H 4250 6825 50  0000 C CNN
 F 1 "RN52" H 4250 6734 50  0000 C CNN
-F 2 "EiMS:RN52" H 3700 6700 50  0001 C CNN
+F 2 "DualEMS_PCB:RN52" H 3700 6700 50  0001 C CNN
 F 3 "" H 3700 6700 50  0001 C CNN
 	1    4250 5650
@@
 $EndComp
 $Comp
-L EiMS:LTC3124 U2
+L DualEMS_PCB:LTC3124 U2
 U 1 1 606E9E02
 P 2900 1250
 F 0 "U2" H 2900 1650 50  0000 C CNN
 F 1 "LTC3124" H 2900 1550 50  0000 C CNN
-F 2 "EiMS:LTC3124" H 2650 1500 50  0001 C CNN
+F 2 "DualEMS_PCB:LTC3124" H 2650 1500 50  0001 C CNN
 F 3 "" H 2650 1500 50  0001 C CNN
 	1    2900 1250
@@
 	2000 2350 2000 2400
 $Comp
-L EiMS:MIWI06-24D05 PS1
+L DualEMS_PCB:MIWI06-24D05 PS1
 U 1 1 6085047C
 P 1450 2750
 F 0 "PS1" V 735 2750 50  0000 C CNN
 F 1 "MIWI06-24D05" V 826 2750 50  0000 C CNN
-F 2 "EiMS:MIWI06-24D05" H 1600 3100 50  0001 C CNN
+F 2 "DualEMS_PCB:MIWI06-24D05" H 1600 3100 50  0001 C CNN
 F 3 "" H 1600 3100 50  0001 C CNN
 	1    1450 2750
@@
 	2000 3450 1900 3450
 $Comp
-L EiMS:LMC662 U3
+L DualEMS_PCB:LMC662 U3
 U 1 1 609796B7
 P 6450 3450
 F 0 "U3" V 6404 3988 50  0000 L CNN
 F 1 "LMC662" V 6495 3988 50  0000 L CNN
-F 2 "EiMS:LMC662" H 5600 4000 50  0001 C CNN
+F 2 "DualEMS_PCB:LMC662" H 5600 4000 50  0001 C CNN
 F 3 "" H 5600 4000 50  0001 C CNN
 	1    6450 3450
@@
 	6300 2150 5000 2150
 $Comp
-L EiMS:IFJM-001 U4
+L DualEMS_PCB:IFJM-001 U4
 U 1 1 60BAFA96
 P 8450 2700
 F 0 "U4" H 8450 3225 50  0000 C CNN
 F 1 "IFJM-001" H 8450 3134 50  0000 C CNN
-F 2 "EiMS:IFJM-001" H 8200 3100 50  0001 C CNN
+F 2 "DualEMS_PCB:IFJM-001" H 8200 3100 50  0001 C CNN
 F 3 "" H 8200 3100 50  0001 C CNN
 	1    8450 2700
@@
 $EndComp
 $Comp
-L EiMS:IFJM-001 U5
+L DualEMS_PCB:IFJM-001 U5
 U 1 1 60BB016D
 P 8450 4800
 F 0 "U5" H 8450 5325 50  0000 C CNN
 F 1 "IFJM-001" H 8450 5234 50  0000 C CNN
-F 2 "EiMS:IFJM-001" H 8200 5200 50  0001 C CNN
+F 2 "DualEMS_PCB:IFJM-001" H 8200 5200 50  0001 C CNN
 F 3 "" H 8200 5200 50  0001 C CNN
 	1    8450 4800
@@
 F 0 "J2" H 11000 2200 50  0000 R CNN
 F 1 "AudioJack2" H 11150 2300 50  0000 R CNN
-F 2 "EiMS:MJ-352" H 10950 2450 50  0001 C CNN
+F 2 "DualEMS_PCB:MJ-352" H 10950 2450 50  0001 C CNN
 F 3 "~" H 10950 2450 50  0001 C CNN
 	1    10950 2450
@@
 F 0 "J3" H 11000 4300 50  0000 R CNN
 F 1 "AudioJack2" H 11150 4400 50  0000 R CNN
-F 2 "EiMS:MJ-352" H 10950 4550 50  0001 C CNN
+F 2 "DualEMS_PCB:MJ-352" H 10950 4550 50  0001 C CNN
 F 3 "~" H 10950 4550 50  0001 C CNN
 	1    10950 4550
@@
 	7450 4950 7750 4950
 $Comp
-L EiMS:M78AR033-0.5 PS2
+L DualEMS_PCB:M78AR033-0.5 PS2
 U 1 1 60871870
 P 1700 4400
 F 0 "PS2" V 1654 4588 50  0000 L CNN
 F 1 "M78AR033-0.5" V 1745 4588 50  0000 L CNN
-F 2 "EiMS:M78AR033-0.5" H 1400 4850 50  0001 C CNN
+F 2 "DualEMS_PCB:M78AR033-0.5" H 1400 4850 50  0001 C CNN
 F 3 "" H 1400 4850 50  0001 C CNN
 	1    1700 4400
@@
 $EndComp
 $Comp
-L EiMS:PIC32MM0064GPL028-I_SP U1
+L DualEMS_PCB:PIC32MM0064GPL028-I_SP U1
 U 1 1 60AD39E9
 P 2100 6100
 F 0 "U1" H 2100 6975 50  0000 C CNN
 F 1 "PIC32MM0064GPL028-I_SP" H 2100 6884 50  0000 C CNN
-F 2 "EiMS:PIC32MM0064GPL028-I_SP" H 1750 6900 50  0001 C CNN
+F 2 "DualEMS_PCB:PIC32MM0064GPL028-I_SP" H 1750 6900 50  0001 C CNN
 F 3 "" H 1750 6900 50  0001 C CNN
 	1    2100 6100
@@
 $EndComp
 $Comp
-L EiMS:+3V7 #PWR03
+L DualEMS_PCB:+3V7 #PWR03
 U 1 1 60886DD0
 P 2050 1000
 F 0 "#PWR03" H 2050 850 50  0001 C CNN
 F 1 "+3V7" H 2065 1173 50  0000 C CNN
-F 2 "" H 1950 1150 50  0001 C CNN
+F 2 "DualEMS_PCB:Battery_+3V7" H 1950 1150 50  0001 C CNN
 F 3 "" H 1950 1150 50  0001 C CNN
 	1    2050 1000
@@
 $EndComp
 $Comp
-L EiMS:+3V7 #PWR01
+L DualEMS_PCB:+3V7 #PWR01
 U 1 1 608988CA
 P 800 1000
 F 0 "#PWR01" H 800 850 50  0001 C CNN
 F 1 "+3V7" H 815 1173 50  0000 C CNN
-F 2 "" H 700 1150 50  0001 C CNN
+F 2 "DualEMS_PCB:Battery_+3V7" H 700 1150 50  0001 C CNN
 F 3 "" H 700 1150 50  0001 C CNN
 	1    800  1000
@@
 F 0 "BT1" H 918 1396 50  0000 L CNN
 F 1 "Battery_Cell" H 918 1305 50  0000 L CNN
-F 2 "EiMS:Battery_+3V7" V 800 1360 50  0001 C CNN
+F 2 "DualEMS_PCB:Battery_+3V7" V 800 1360 50  0001 C CNN
 F 3 "~" V 800 1360 50  0001 C CNN
 	1    800  1300
