File: DualEMS_PCB.kicad_pcb (KiCad board)
At the start: 4 copper layers, 200 x 123 mm, 62 parts, among them J1 Conn_01x06, J2 AudioJack2, J3 AudioJack2, SW1 SW_SPDT, U1 PIC32MM0064GPL028-I_SP, U2 LTC3124, U3 LMC662, U4 IFJM-001, U5 IFJM-001

Commit message: updated for kiCad 6.0
Other:
- net class Default removed
- net class Power_12 removed
- net class Power_3.3 removed
- net class Power_3.7 removed
- net class Power_5 removed
- net class Power_GND0 removed
- net class Power_GND1 removed
- net class Signal_Analog removed
- net class Signal_Digital removed
